Commit message: update on travel_mount

File: src/cyclus_description/urdf/emrac_body.urdf.xacro (robot description, xacro)
@@ -1,5 +1,5 @@
 <robot name="emrac_body" xmlns:xacro="http://www.ros.org/wiki/xacro">
   <xacro:property name="lift_plate_scale" value="0.001 0.001 0.001" />
-  <xacro:property name="lift_plate_mount_y" value="-0.32" />
+  <xacro:property name="lift_plate_mount_y" value="-1.05" />
   <xacro:property name="lift_plate_travel" value="0.35" />
   <xacro:property name="lift_plate_origin_x" value="-1.90140869140626" />
@@ -95,5 +95,5 @@
   </link>
   <joint name="arm_joint_1" type="revolute">
-    <origin xyz="1.53958467822174 0.780045273498867 -0.0905675614190252" rpy="-1.57079632679425 0 -3.14159265358979" />
+    <origin xyz="1.53958467822174 0.780045273498867 -0.0905675614190252" rpy="-0.78539816339 0 -3.14159265358979" />
     <parent link="docking_1" />
     <child link="dock_arm_1" />
@@ -153,5 +153,5 @@
   </link>
   <joint name="arm_joint_2" type="revolute">
-    <origin xyz="1.50831912172871 0.822636592430764 -0.094403978789434" rpy="0 0 0" />
+    <origin xyz="1.50831912172871 0.822636592430764 -0.094403978789434" rpy="-0.7853981633974483 0 0" />
     <parent link="docking_2" />
     <child link="dock_arm_2" />
@@ -211,5 +211,5 @@
   </link>
   <joint name="arm_joint_3" type="revolute">
-    <origin xyz="2.58061469903853 0.821037736652904 -0.0923428786138167" rpy="0 0 -3.14158674425948" />
+    <origin xyz="2.58061469903853 0.821037736652904 -0.0923428786138167" rpy="-0.7853981633974483 0 -3.14158674425948" />
     <parent link="docking_3" />
     <child link="dock_arm_3" />
@@ -269,5 +269,5 @@
   </link>
   <joint name="arm_joint_4" type="revolute">
-    <origin xyz="0.468826677599663 0.82263659243076 -0.0944039787894324" rpy="0 0 -3.14158674425949" />
+    <origin xyz="0.468826677599663 0.82263659243076 -0.0944039787894324" rpy="-0.7853981633974483 0 -3.14158674425949" />
     <parent link="docking_4" />
     <child link="dock_arm_4" />
@@ -353,10 +353,14 @@
   </gazebo>
   <gazebo reference="lift_plate_carrier">
-    <gravity>false</gravity>
+    <gravity>true</gravity>
     <self_collide>false</self_collide>
   </gazebo>
   <gazebo reference="lift_plate">
-    <gravity>false</gravity>
-    <self_collide>false</self_collide>
-  </gazebo>
+    <gravity>true</gravity>
+    <self_collide>false</self_collide>
+  </gazebo>
+  <gazebo reference="lift_plate">
+  <mu1>1.0</mu1>
+  <mu2>1.0</mu2>
+</gazebo>
 </robot>

Commit message: update_on_final_emrac_pos

File: src/cyclus_description/urdf/emrac_body.urdf.xacro (robot description, xacro)
@@ -1,6 +1,6 @@
 <robot name="emrac_body" xmlns:xacro="http://www.ros.org/wiki/xacro">
   <xacro:property name="lift_plate_scale" value="0.001 0.001 0.001" />
-  <xacro:property name="lift_plate_mount_y" value="-1.05" />
-  <xacro:property name="lift_plate_travel" value="0.35" />
+  <xacro:property name="lift_plate_mount_y" value="-0.29" />
+  <xacro:property name="lift_plate_travel" value="0.6" />
   <xacro:property name="lift_plate_origin_x" value="-1.90140869140626" />
   <xacro:property name="lift_plate_origin_y" value="-0.40512716674804685857" />
@@ -95,6 +95,5 @@
   </link>
   <joint name="arm_joint_1" type="revolute">
-    <origin xyz="1.53958467822174 0.780045273498867 -0.0905675614190252" rpy="-0.78539816339 0 -3.14159265358979" />
-    <parent link="docking_1" />
+    <origin xyz="1.53958467822174 0.780045273498867 -0.0905675614190252" rpy="-1.57079632679425 0 -3.14159265358979" />    <parent link="docking_1" />
     <child link="dock_arm_1" />
     <axis xyz="-1 0 0" />
@@ -153,5 +152,5 @@
   </link>
   <joint name="arm_joint_2" type="revolute">
-    <origin xyz="1.50831912172871 0.822636592430764 -0.094403978789434" rpy="-0.7853981633974483 0 0" />
+    <origin xyz="1.50831912172871 0.822636592430764 -0.094403978789434" rpy="0 0 0" />
     <parent link="docking_2" />
     <child link="dock_arm_2" />
@@ -211,5 +210,5 @@
   </link>
   <joint name="arm_joint_3" type="revolute">
-    <origin xyz="2.58061469903853 0.821037736652904 -0.0923428786138167" rpy="-0.7853981633974483 0 -3.14158674425948" />
+    <origin xyz="2.58061469903853 0.821037736652904 -0.0923428786138167" rpy="0 0 -3.14158674425948" />
     <parent link="docking_3" />
     <child link="dock_arm_3" />
@@ -269,5 +268,5 @@
   </link>
   <joint name="arm_joint_4" type="revolute">
-    <origin xyz="0.468826677599663 0.82263659243076 -0.0944039787894324" rpy="-0.7853981633974483 0 -3.14158674425949" />
+    <origin xyz="0.468826677599663 0.82263659243076 -0.0944039787894324" rpy="0 0 -3.14158674425949" />
     <parent link="docking_4" />
     <child link="dock_arm_4" />
@@ -308,5 +307,5 @@
     <child link="lift_plate_carrier" />
     <axis xyz="0 -1 0" />
-    <limit lower="-${lift_plate_travel}" upper="${lift_plate_travel}" effort="500.0" velocity="0.15" />
+    <limit lower="0.0" upper="${lift_plate_travel}" effort="500.0" velocity="0.15" />
     <dynamics damping="30.0" friction="10.0" />
   </joint>

Commit message: fixed the emrac movements

File: src/cyclus_description/urdf/emrac_body.urdf.xacro (robot description, xacro)
@@ -2,11 +2,20 @@
   <xacro:property name="lift_plate_scale" value="0.001 0.001 0.001" />
   <xacro:property name="lift_plate_mount_y" value="-0.29" />
-  <xacro:property name="lift_plate_travel" value="0.6" />
+  <xacro:property name="lift_plate_travel" value="0.4" />
   <xacro:property name="lift_plate_origin_x" value="-1.90140869140626" />
   <xacro:property name="lift_plate_origin_y" value="-0.40512716674804685857" />
   <xacro:property name="lift_plate_origin_z" value="0.45429059314727783" />
   <xacro:property name="lift_plate_roll" value="1.5707963267949" />
+  <xacro:property name="lift_plate_collision_size" value="1.02 0.66 0.03" />
+  <xacro:property name="dock_arm_collision_length" value="0.78" />
+  <xacro:property name="dock_arm_collision_radius" value="0.02" />
   <material name="lift_plate_grey">
     <color rgba="0.72 0.72 0.72 1.0" />
+  </material>
+  <material name="carrier_charcoal">
+    <color rgba="0.22 0.23 0.24 1.0" />
+  </material>
+  <material name="carrier_black">
+    <color rgba="0.14 0.14 0.15 1.0" />
   </material>
   <link name="emrac_body_root">
@@ -33,7 +42,5 @@
         <mesh filename="file:///home/bargavan/cyclus/src/carrier_emrac/meshes/visual/base_link.STL" />
       </geometry>
-      <material name="">
-        <color rgba="0.529411764705882 0.549019607843137 0.549019607843137 1" />
-      </material>
+      <material name="carrier_charcoal" />
     </visual>
     <collision>
@@ -55,7 +62,5 @@
         <mesh filename="file:///home/bargavan/cyclus/src/carrier_emrac/meshes/visual/docking_1.STL" />
       </geometry>
-      <material name="">
-        <color rgba="0.792156862745098 0.819607843137255 0.933333333333333 1" />
-      </material>
+      <material name="carrier_black" />
     </visual>
     <collision>
@@ -83,20 +88,19 @@
         <mesh filename="file:///home/bargavan/cyclus/src/carrier_emrac/meshes/visual/dock_arm_1.STL" />
       </geometry>
-      <material name="">
-        <color rgba="0.792156862745098 0.819607843137255 0.933333333333333 1" />
-      </material>
-    </visual>
-    <collision>
-      <origin xyz="0 0 0" rpy="0 0 0" />
-      <geometry>
-        <mesh filename="file:///home/bargavan/cyclus/src/carrier_emrac/meshes/collision/dock_arm_1.STL" />
+      <material name="carrier_black" />
+    </visual>
+    <collision>
+      <origin xyz="0.39 0 0" rpy="0 1.5707963267949 0" />
+      <geometry>
+        <cylinder radius="${dock_arm_collision_radius}" length="${dock_arm_collision_length}" />
       </geometry>
     </collision>
   </link>
   <joint name="arm_joint_1" type="revolute">
-    <origin xyz="1.53958467822174 0.780045273498867 -0.0905675614190252" rpy="-1.57079632679425 0 -3.14159265358979" />    <parent link="docking_1" />
+    <origin xyz="1.53958467822174 0.780045273498867 -0.0905675614190252" rpy="-1.57079632679425 0 -3.14159265358979" />
+    <parent link="docking_1" />
     <child link="dock_arm_1" />
     <axis xyz="-1 0 0" />
-    <limit lower="-0.78539816339" upper="0.78539816339" effort="200.0" velocity="0.2" />
+    <limit lower="-0.78539816339" upper="0.78539816339" effort="200.0" velocity="1.0" />
     <dynamics damping="50.0" friction="20.0" />
   </joint>
@@ -112,7 +116,5 @@
         <mesh filename="file:///home/bargavan/cyclus/src/carrier_emrac/meshes/visual/docking_2.STL" />
       </geometry>
-      <material name="">
-        <color rgba="0.792156862745098 0.819607843137255 0.933333333333333 1" />
-      </material>
+      <material name="carrier_black" />
     </visual>
     <collision>
@@ -140,12 +142,10 @@
         <mesh filename="file:///home/bargavan/cyclus/src/carrier_emrac/meshes/visual/dock_arm_2.STL" />
       </geometry>
-      <material name="">
-        <color rgba="0.792156862745098 0.819607843137255 0.933333333333333 1" />
-      </material>
-    </visual>
-    <collision>
-      <origin xyz="0 0 0" rpy="0 0 0" />
-      <geometry>
-        <mesh filename="file:///home/bargavan/cyclus/src/carrier_emrac/meshes/collision/dock_arm_2.STL" />
+      <material name="carrier_black" />
+    </visual>
+    <collision>
+      <origin xyz="0.39 0 0" rpy="0 1.5707963267949 0" />
+      <geometry>
+        <cylinder radius="${dock_arm_collision_radius}" length="${dock_arm_collision_length}" />
       </geometry>
     </collision>
@@ -156,5 +156,5 @@
     <child link="dock_arm_2" />
     <axis xyz="1 0 0" />
-    <limit lower="-0.78539816339" upper="0.78539816339" effort="200.0" velocity="0.2" />
+    <limit lower="-0.78539816339" upper="0.78539816339" effort="200.0" velocity="1.0" />
     <dynamics damping="50.0" friction="20.0" />
   </joint>
@@ -170,7 +170,5 @@
         <mesh filename="file:///home/bargavan/cyclus/src/carrier_emrac/meshes/visual/docking_3.STL" />
       </geometry>
-      <material name="">
-        <color rgba="0.792156862745098 0.819607843137255 0.933333333333333 1" />
-      </material>
+      <material name="carrier_black" />
     </visual>
     <collision>
@@ -198,12 +196,10 @@
         <mesh filename="file:///home/bargavan/cyclus/src/carrier_emrac/meshes/visual/dock_arm_3.STL" />
       </geometry>
-      <material name="">
-        <color rgba="0.792156862745098 0.819607843137255 0.933333333333333 1" />
-      </material>
-    </visual>
-    <collision>
-      <origin xyz="0 0 0" rpy="0 0 0" />
-      <geometry>
-        <mesh filename="file:///home/bargavan/cyclus/src/carrier_emrac/meshes/collision/dock_arm_3.STL" />
+      <material name="carrier_black" />
+    </visual>
+    <collision>
+      <origin xyz="-0.39 0 0" rpy="0 1.5707963267949 0" />
+      <geometry>
+        <cylinder radius="${dock_arm_collision_radius}" length="${dock_arm_collision_length}" />
       </geometry>
     </collision>
@@ -214,5 +210,5 @@
     <child link="dock_arm_3" />
     <axis xyz="-0.99999999998254 0 0" />
-    <limit lower="-0.78539816339" upper="0.78539816339" effort="200.0" velocity="0.2" />
+    <limit lower="-0.78539816339" upper="0.78539816339" effort="200.0" velocity="1.0" />
     <dynamics damping="50.0" friction="20.0" />
   </joint>
@@ -228,7 +224,5 @@
         <mesh filename="file:///home/bargavan/cyclus/src/carrier_emrac/meshes/visual/docking_4.STL" />
       </geometry>
-      <material name="">
-        <color rgba="0.792156862745098 0.819607843137255 0.933333333333333 1" />
-      </material>
+      <material name="carrier_black" />
     </visual>
     <collision>
@@ -256,12 +250,10 @@
         <mesh filename="file:///home/bargavan/cyclus/src/carrier_emrac/meshes/visual/dock_arm_4.STL" />
       </geometry>
-      <material name="">
-        <color rgba="0.792156862745098 0.819607843137255 0.933333333333333 1" />
-      </material>
-    </visual>
-    <collision>
-      <origin xyz="0 0 0" rpy="0 0 0" />
-      <geometry>
-        <mesh filename="file:///home/bargavan/cyclus/src/carrier_emrac/meshes/collision/dock_arm_4.STL" />
+      <material name="carrier_black" />
+    </visual>
+    <collision>
+      <origin xyz="-0.39 0 0" rpy="0 1.5707963267949 0" />
+      <geometry>
+        <cylinder radius="${dock_arm_collision_radius}" length="${dock_arm_collision_length}" />
       </geometry>
     </collision>
@@ -272,5 +264,5 @@
     <child link="dock_arm_4" />
     <axis xyz="0.99999999998254 0 0" />
-    <limit lower="-0.78539816339" upper="0.78539816339" effort="200.0" velocity="0.2" />
+    <limit lower="-0.78539816339" upper="0.78539816339" effort="200.0" velocity="1.0" />
     <dynamics damping="50.0" friction="20.0" />
   </joint>
@@ -298,5 +290,5 @@
       <origin xyz="${lift_plate_origin_x} ${lift_plate_origin_y} ${lift_plate_origin_z}" rpy="${lift_plate_roll} 0 0" />
       <geometry>
-        <mesh filename="file://$(find cyclus_description)/meshes/emrac/EMRAC Lift Plate Dwn Pos 1.stl" scale="${lift_plate_scale}" />
+        <box size="${lift_plate_collision_size}" />
       </geometry>
     </collision>
@@ -307,6 +299,6 @@
     <child link="lift_plate_carrier" />
     <axis xyz="0 -1 0" />
-    <limit lower="0.0" upper="${lift_plate_travel}" effort="500.0" velocity="0.15" />
-    <dynamics damping="30.0" friction="10.0" />
+    <limit lower="-${lift_plate_travel}" upper="${lift_plate_travel}" effort="1000.0" velocity="0.58" />
+    <dynamics damping="1.0" friction="0.05" />
   </joint>
   <joint name="lift_plate_mount" type="fixed">
@@ -315,39 +307,93 @@
     <child link="lift_plate" />
   </joint>
+  <ros2_control name="GazeboSimSystem" type="system">
+    <hardware>
+      <plugin>gz_ros2_control/GazeboSimSystem</plugin>
+    </hardware>
+    <joint name="base_to_lift_plate_carrier">
+      <command_interface name="position" />
+      <state_interface name="position" />
+      <state_interface name="velocity" />
+    </joint>
+    <joint name="arm_joint_1">
+      <command_interface name="position" />
+      <state_interface name="position" />
+      <state_interface name="velocity" />
+    </joint>
+    <joint name="arm_joint_2">
+      <command_interface name="position" />
+      <state_interface name="position" />
+      <state_interface name="velocity" />
+    </joint>
+    <joint name="arm_joint_3">
+      <command_interface name="position" />
+      <state_interface name="position" />
+      <state_interface name="velocity" />
+    </joint>
+    <joint name="arm_joint_4">
+      <command_interface name="position" />
+      <state_interface name="position" />
+      <state_interface name="velocity" />
+    </joint>
+  </ros2_control>
+  <gazebo>
+    <self_collide>true</self_collide>
+    <plugin filename="libgz_ros2_control-system.so" name="gz_ros2_control::GazeboSimROS2ControlPlugin">
+      <parameters>$(find cyclus_description)/config/emrac_arm_controllers.yaml</parameters>
+      <controller_manager_node_name>controller_manager</controller_manager_node_name>
+    </plugin>
+  </gazebo>
   <gazebo reference="base_link">
+    <material>Gazebo/DarkGrey</material>
     <gravity>false</gravity>
     <self_collide>false</self_collide>
   </gazebo>
   <gazebo reference="docking_1">
+    <material>Gazebo/Black</material>
     <gravity>false</gravity>
     <self_collide>false</self_collide>
   </gazebo>
   <gazebo reference="dock_arm_1">
-    <gravity>false</gravity>
-    <self_collide>false</self_collide>
+    <material>Gazebo/Black</material>
+    <gravity>false</gravity>
+    <self_collide>true</self_collide>
+    <mu1>2.0</mu1>
+    <mu2>2.0</mu2>
   </gazebo>
   <gazebo reference="docking_2">
+    <material>Gazebo/Black</material>
     <gravity>false</gravity>
     <self_collide>false</self_collide>
   </gazebo>
   <gazebo reference="dock_arm_2">
-    <gravity>false</gravity>
-    <self_collide>false</self_collide>
+    <material>Gazebo/Black</material>
+    <gravity>false</gravity>
+    <self_collide>true</self_collide>
+    <mu1>2.0</mu1>
+    <mu2>2.0</mu2>
   </gazebo>
   <gazebo reference="docking_3">
+    <material>Gazebo/Black</material>
     <gravity>false</gravity>
     <self_collide>false</self_collide>
   </gazebo>
   <gazebo reference="dock_arm_3">
-    <gravity>false</gravity>
-    <self_collide>false</self_collide>
+    <material>Gazebo/Black</material>
+    <gravity>false</gravity>
+    <self_collide>true</self_collide>
+    <mu1>2.0</mu1>
+    <mu2>2.0</mu2>
   </gazebo>
   <gazebo reference="docking_4">
+    <material>Gazebo/Black</material>
     <gravity>false</gravity>
     <self_collide>false</self_collide>
   </gazebo>
   <gazebo reference="dock_arm_4">
-    <gravity>false</gravity>
-    <self_collide>false</self_collide>
+    <material>Gazebo/Black</material>
+    <gravity>false</gravity>
+    <self_collide>true</self_collide>
+    <mu1>2.0</mu1>
+    <mu2>2.0</mu2>
   </gazebo>
   <gazebo reference="lift_plate_carrier">
@@ -356,10 +402,9 @@
   </gazebo>
   <gazebo reference="lift_plate">
+    <material>Gazebo/LightGrey</material>
     <gravity>true</gravity>
-    <self_collide>false</self_collide>
-  </gazebo>
-  <gazebo reference="lift_plate">
-  <mu1>1.0</mu1>
-  <mu2>1.0</mu2>
-</gazebo>
+    <self_collide>true</self_collide>
+    <mu1>2.0</mu1>
+    <mu2>2.0</mu2>
+  </gazebo>
 </robot>
