Commit message: EMRAC_4 INTEGRATION

File: src/cyclus_description/urdf/cyclus_integrated_system.urdf.xacro (robot description, xacro)
@@ -1,8 +1,9 @@
 <robot name="cyclus_integrated_system" xmlns:xacro="http://www.ros.org/wiki/xacro">
+  <xacro:include filename="/home/bargavan/cyclus/src/cyclus_description/urdf/emrac_body_macro.xacro" />
   <xacro:arg name="structure_gap_mm" default="1960.0" />
   <xacro:arg name="stationary_z_offset" default="0.5" />
   <xacro:arg name="ground_rails_mount_x" default="1.9" />
   <xacro:arg name="ground_rails_mount_y" default="-0.02" />
-  <xacro:arg name="ground_rails_mount_z" default="0.3" />
+  <xacro:arg name="ground_rails_mount_z" default="0.5" />
   <xacro:arg name="emrac_axis_1_xyz" default="1,0,0" />
   <xacro:arg name="emrac_axis_2_xyz" default="0,0,-1" />
@@ -11,5 +12,6 @@
   <xacro:arg name="emrac_mount_x" default="0.95" />
   <xacro:arg name="emrac_mount_y" default="0.47" />
-  <xacro:arg name="emrac_mount_z" default="0.0" />
+  <xacro:arg name="emrac_mount_z" default="0.3" />
+  <xacro:arg name="emrac_stack_z_step" default="0.5" />
   <xacro:property name="mesh_scale" value="0.001 0.001 0.001" />
   <xacro:property name="stationary_mesh_roll" value="0.0" />
@@ -33,30 +35,17 @@
   <xacro:property name="emrac_axis_1_vector" value="${' '.join('$(arg emrac_axis_1_xyz)'.split(','))}" />
   <xacro:property name="emrac_axis_2_vector" value="${' '.join('$(arg emrac_axis_2_xyz)'.split(','))}" />
-  <xacro:property name="lift_plate_scale" value="0.001 0.001 0.001" />
-  <xacro:property name="lift_plate_mount_y" value="-0.29" />
-  <xacro:property name="lift_plate_travel" value="0.4" />
-  <xacro:property name="lift_plate_origin_x" value="-1.90140869140626" />
-  <xacro:property name="lift_plate_origin_y" value="-0.40512716674804685857" />
-  <xacro:property name="lift_plate_origin_z" value="0.45429059314727783" />
-  <xacro:property name="lift_plate_roll" value="1.5707963267949" />
-  <xacro:property name="lift_plate_collision_size" value="1.02 0.66 0.03" />
-  <xacro:property name="dock_arm_collision_length" value="0.78" />
-  <xacro:property name="dock_arm_collision_radius" value="0.02" />
-  <xacro:property name="base_collision_origin" value="0.1927191019 -0.6836163700 0.4518507421" />
-  <xacro:property name="base_collision_size" value="1.4354550838 0.2207220197 2.1443541646" />
-  <xacro:property name="docking_collision_origin" value="1.5734563470 0.7781362534 -0.0910039619" />
-  <xacro:property name="docking_collision_origin_2" value="1.5736307502 0.8207275867 -0.0948403776" />
-  <xacro:property name="docking_collision_size" value="0.0677434206 0.0609734058 0.0491782576" />
-  <material name="lift_plate_grey">
-    <color rgba="0.72 0.72 0.72 1.0" />
+  <xacro:property name="emrac_mount_z_value" value="$(arg emrac_mount_z)" />
+  <xacro:property name="emrac_stack_z_step_value" value="$(arg emrac_stack_z_step)" />
+  <material name="steel_frame">
+    <color rgba="0.25 0.25 0.25 1.0" />
   </material>
   <material name="carrier_charcoal">
-    <color rgba="0.22 0.23 0.24 1.0" />
+    <color rgba="0.36 0.38 0.40 1.0" />
   </material>
   <material name="carrier_black">
-    <color rgba="0.14 0.14 0.15 1.0" />
+    <color rgba="0.24 0.25 0.27 1.0" />
   </material>
-  <material name="steel_frame">
-    <color rgba="0.25 0.25 0.25 1.0" />
+  <material name="lift_plate_grey">
+    <color rgba="0.78 0.78 0.76 1.0" />
   </material>
   <link name="world" />
@@ -68,4 +57,9 @@
     </inertial>
   </link>
+  <joint name="world_to_integrated_root" type="fixed">
+    <parent link="world" />
+    <child link="integrated_root" />
+    <origin xyz="0 0 0" rpy="0 0 0" />
+  </joint>
   <link name="stationary_structure_right">
     <inertial>
@@ -143,372 +137,194 @@
     <origin xyz="$(arg ground_rails_mount_x) $(arg ground_rails_mount_y) $(arg ground_rails_mount_z)" rpy="0 0 0" />
   </joint>
-  <joint name="world_to_integrated_root" type="fixed">
-    <parent link="world" />
-    <child link="integrated_root" />
-    <origin xyz="0 0 0" rpy="0 0 0" />
-  </joint>
-  <link name="emrac_axis_1_carrier">
-    <inertial>
+  <xacro:macro name="emrac_planar_mount" params="prefix mount_z">
+    <link name="${prefix}slide_axis_1_carrier">
+      <inertial>
+        <origin xyz="0 0 0" rpy="0 0 0" />
+        <mass value="0.1" />
+        <inertia ixx="1e-3" ixy="0" ixz="0" iyy="1e-3" iyz="0" izz="1e-3" />
+      </inertial>
+    </link>
+    <link name="${prefix}slide_axis_2_carrier">
+      <inertial>
+        <origin xyz="0 0 0" rpy="0 0 0" />
+        <mass value="0.1" />
+        <inertia ixx="1e-3" ixy="0" ixz="0" iyy="1e-3" iyz="0" izz="1e-3" />
+      </inertial>
+    </link>
+    <joint name="${prefix}slide_axis_1" type="prismatic">
+      <origin xyz="$(arg emrac_mount_x) $(arg emrac_mount_y) ${mount_z}" rpy="0 0 0" />
+      <parent link="integrated_root" />
+      <child link="${prefix}slide_axis_1_carrier" />
+      <axis xyz="${emrac_axis_1_vector}" />
+      <limit lower="-${emrac_axis_1_limit}" upper="${emrac_axis_1_limit}" effort="50000.0" velocity="2.0" />
+      <dynamics damping="0.5" friction="0.0" />
+    </joint>
+    <joint name="${prefix}slide_axis_2" type="prismatic">
       <origin xyz="0 0 0" rpy="0 0 0" />
-      <mass value="0.1" />
-      <inertia ixx="1e-3" ixy="0" ixz="0" iyy="1e-3" iyz="0" izz="1e-3" />
-    </inertial>
-  </link>
-  <link name="emrac_axis_2_carrier">
-    <inertial>
+      <parent link="${prefix}slide_axis_1_carrier" />
+      <child link="${prefix}slide_axis_2_carrier" />
+      <axis xyz="${emrac_axis_2_vector}" />
+      <limit lower="-${emrac_axis_2_limit}" upper="${emrac_axis_2_limit}" effort="50000.0" velocity="2.0" />
+      <dynamics damping="0.5" friction="0.0" />
+    </joint>
+    <xacro:emrac_body_instance prefix="${prefix}" />
+    <joint name="${prefix}slide_axis_2_to_body_root" type="fixed">
       <origin xyz="0 0 0" rpy="0 0 0" />
-      <mass value="0.1" />
-      <inertia ixx="1e-3" ixy="0" ixz="0" iyy="1e-3" iyz="0" izz="1e-3" />
-    </inertial>
-  </link>
-  <joint name="emrac_slide_axis_1" type="prismatic">
-    <origin xyz="$(arg emrac_mount_x) $(arg emrac_mount_y) $(arg emrac_mount_z)" rpy="0 0 0" />
-    <parent link="integrated_root" />
-    <child link="emrac_axis_1_carrier" />
-    <axis xyz="${emrac_axis_1_vector}" />
-    <limit lower="-${emrac_axis_1_limit}" upper="${emrac_axis_1_limit}" effort="50000.0" velocity="2.0" />
-    <dynamics damping="0.5" friction="0.0" />
-  </joint>
-  <joint name="emrac_slide_axis_2" type="prismatic">
-    <origin xyz="0 0 0" rpy="0 0 0" />
-    <parent link="emrac_axis_1_carrier" />
-    <child link="emrac_axis_2_carrier" />
-    <axis xyz="${emrac_axis_2_vector}" />
-    <limit lower="-${emrac_axis_2_limit}" upper="${emrac_axis_2_limit}" effort="50000.0" velocity="2.0" />
-    <dynamics damping="0.5" friction="0.0" />
-  </joint>
-  <link name="emrac_body_root">
-    <inertial>
-      <origin xyz="0 0 0" rpy="0 0 0" />
-      <mass value="0.001" />
-      <inertia ixx="1e-6" ixy="0" ixz="0" iyy="1e-6" iyz="0" izz="1e-6" />
-    </inertial>
-  </link>
-  <joint name="emrac_axis_2_to_body_root" type="fixed">
-    <origin xyz="0 0 0" rpy="0 0 0" />
-    <parent link="emrac_axis_2_carrier" />
-    <child link="emrac_body_root" />
-  </joint>
-  <joint name="emrac_body_root_to_base_link" type="fixed">
-    <origin xyz="0 0 0" rpy="-1.5707963267949 0 3.14159265358979" />
-    <parent link="emrac_body_root" />
-    <child link="base_link" />
-  </joint>
-  <link name="base_link">
-    <inertial>
-      <origin xyz="0.231326122438629 -0.729625066059866 -0.384275142354278" rpy="0 0 0" />
-      <mass value="66.8400447533962" />
-      <inertia ixx="0.126647867330863" ixy="1.09468303143366E-14" ixz="1.49222860415562E-14" iyy="0.489903098665309" iyz="-7.74690196420397E-11" izz="0.480399430509725" />
-    </inertial>
-    <visual>
-      <origin xyz="0 0 0" rpy="0 0 0" />
-      <geometry>
-        <mesh filename="file:///home/bargavan/cyclus/src/carrier_emrac/meshes/visual/base_link.STL" />
-      </geometry>
-      <material name="carrier_charcoal" />
-    </visual>
-    <collision>
-      <origin xyz="${base_collision_origin}" rpy="0 0 0" />
-      <geometry>
-        <box size="${base_collision_size}" />
-      </geometry>
-    </collision>
-  </link>
-  <link name="docking_1">
-    <inertial>
-      <origin xyz="1.57308467822174 0.780045273498867 -0.0905675614190253" rpy="0 0 0" />
-      <mass value="0.0202336294869927" />
-      <inertia ixx="9.72507400857707E-07" ixy="-2.37554290260085E-20" ixz="1.13271025171526E-20" iyy="8.0553172643547E-06" iyz="3.70971200079535E-35" izz="8.0553172643547E-06" />
-    </inertial>
-    <visual>
-      <origin xyz="0 0 0" rpy="0 0 0" />
-      <geometry>
-        <mesh filename="file:///home/bargavan/cyclus/src/carrier_emrac/meshes/visual/docking_1.STL" />
-      </geometry>
-      <material name="carrier_black" />
-    </visual>
-    <collision>
-      <origin xyz="${docking_collision_origin}" rpy="0 0 0" />
-      <geometry>
-        <box size="${docking_collision_size}" />
-      </geometry>
-    </collision>
-  </link>
-  <joint name="dock_joint_1" type="fixed">
-    <origin xyz="-1.90167019372611 -0.688928868898414 0.456357618202888" rpy="1.5707963267949 0 0" />
-    <parent link="base_link" />
-    <child link="docking_1" />
-    <axis xyz="0 0 0" />
-  </joint>
-  <link name="dock_arm_1">
-    <inertial>
-      <origin xyz="-0.000499999999999778 -0.000407762481728469 -0.000569115410858689" rpy="0 0 0" />
-      <mass value="0.00150072453201757" />
-      <inertia ixx="5.7113098325987E-07" ixy="-2.09373257761955E-22" ixz="-9.42175268372246E-22" iyy="3.76033847997044E-07" iyz="6.32661441841782E-11" izz="1.95347256018162E-07" />
-    </inertial>
-    <visual>
-      <origin xyz="0 0 0" rpy="0 0 0" />
-      <geometry>
-        <mesh filename="file:///home/bargavan/cyclus/src/carrier_emrac/meshes/visual/dock_arm_1.STL" />
-      </geometry>
-      <material name="carrier_black" />
-    </visual>
-    <collision>
-      <origin xyz="0.39 0 0" rpy="0 1.5707963267949 0" />
-      <geometry>
-        <cylinder radius="${dock_arm_collision_radius}" length="${dock_arm_collision_length}" />
-      </geometry>
-    </collision>
-  </link>
-  <joint name="arm_joint_1" type="revolute">
-    <origin xyz="1.53958467822174 0.780045273498867 -0.0905675614190252" rpy="-1.57079632679425 0 -3.14159265358979" />
-    <parent link="docking_1" />
-    <child link="dock_arm_1" />
-    <axis xyz="-1 0 0" />
-    <limit lower="-0.78539816339" upper="0.78539816339" effort="200.0" velocity="1.0" />
-    <dynamics damping="50.0" friction="20.0" />
-  </joint>
-  <link name="docking_2">
-    <inertial>
-      <origin xyz="1.57325903320313 0.822636592430764 -0.0944039787894341" rpy="0 0 0" />
-      <mass value="0.0202336294869927" />
-      <inertia ixx="9.72507400857707E-07" ixy="-2.37554290260085E-20" ixz="1.13271025171526E-20" iyy="8.0553172643547E-06" iyz="3.90082702343961E-35" izz="8.0553172643547E-06" />
-    </inertial>
-    <visual>
-      <origin xyz="0 0 0" rpy="0 0 0" />
-      <geometry>
-        <mesh filename="file:///home/bargavan/cyclus/src/carrier_emrac/meshes/visual/docking_2.STL" />
-      </geometry>
-      <material name="carrier_black" />
-    </visual>
-    <collision>
-      <origin xyz="${docking_collision_origin_2}" rpy="0 0 0" />
-      <geometry>
-        <box size="${docking_collision_size}" />
-      </geometry>
-    </collision>
-  </link>
-  <joint name="docking_joint_2" type="fixed">
-    <origin xyz="-0.85761797977807 -0.693687257483896 0.414480042632792" rpy="1.5707963267949 0 0" />
-    <parent link="base_link" />
-    <child link="docking_2" />
-    <axis xyz="1 0 0" />
-  </joint>
-  <link name="dock_arm_2">
-    <inertial>
-      <origin xyz="0.030939911474413 0.000569115410858911 0.000407762481728025" rpy="0 0 0" />
-      <mass value="0.00150072453201757" />
-      <inertia ixx="5.7113098325987E-07" ixy="6.42213640349087E-22" ixz="1.33311741135265E-22" iyy="1.95347256018162E-07" iyz="6.32661443007841E-11" izz="3.76033847997044E-07" />
-    </inertial>
-    <visual>
-      <origin xyz="0 0 0" rpy="0 0 0" />
-      <geometry>
-        <mesh filename="file:///home/bargavan/cyclus/src/carrier_emrac/meshes/visual/dock_arm_2.STL" />
-      </geometry>
-      <material name="carrier_black" />
-    </visual>
-    <collision>
-      <origin xyz="0.39 0 0" rpy="0 1.5707963267949 0" />
-      <geometry>
-        <cylinder radius="${dock_arm_collision_radius}" length="${dock_arm_collision_length}" />
-      </geometry>
-    </collision>
-  </link>
-  <joint name="arm_joint_2" type="revolute">
-    <origin xyz="1.50831912172871 0.822636592430764 -0.094403978789434" rpy="0 0 0" />
-    <parent link="docking_2" />
-    <child link="dock_arm_2" />
-    <axis xyz="1 0 0" />
-    <limit lower="-0.78539816339" upper="0.78539816339" effort="200.0" velocity="1.0" />
-    <dynamics damping="50.0" friction="20.0" />
-  </joint>
-  <link name="docking_3">
-    <inertial>
-      <origin xyz="1.57325903320313 0.822636592430764 -0.0944039787894342" rpy="0 0 0" />
-      <mass value="0.0202336294869927" />
-      <inertia ixx="9.72507400857707E-07" ixy="-2.37554290260085E-20" ixz="1.13271025171526E-20" iyy="8.0553172643547E-06" iyz="3.78249840438576E-35" izz="8.0553172643547E-06" />
-    </inertial>
-    <visual>
-      <origin xyz="0 0 0" rpy="0 0 0" />
-      <geometry>
-        <mesh filename="file:///home/bargavan/cyclus/src/carrier_emrac/meshes/visual/docking_3.STL" />
-      </geometry>
-      <material name="carrier_black" />
-    </visual>
-    <collision>
-      <origin xyz="${docking_collision_origin_2}" rpy="0 0 0" />
-      <geometry>
-        <box size="${docking_collision_size}" />
-      </geometry>
-    </collision>
-  </link>
-  <joint name="docking_joint_3" type="fixed">
-    <origin xyz="-1.89847364561348 -0.683810169290989 -1.15695984220038" rpy="1.5707963267949 0 0" />
-    <parent link="base_link" />
-    <child link="docking_3" />
-    <axis xyz="0 0 0" />
-  </joint>
-  <link name="dock_arm_3">
-    <inertial>
-      <origin xyz="0.974355659733319 -0.00103549815645604 -0.00165333769388842" rpy="0 0 0" />
-      <mass value="0.00150072453201743" />
-      <inertia ixx="5.71130983246695E-07" ixy="-2.2206301702031E-12" ixz="3.7386126927141E-16" iyy="1.95347256031264E-07" iyz="6.32661442999355E-11" izz="3.76033847997012E-07" />
-    </inertial>
-    <visual>
-      <origin xyz="0 0 0" rpy="0 0 0" />
-      <geometry>
-        <mesh filename="file:///home/bargavan/cyclus/src/carrier_emrac/meshes/visual/dock_arm_3.STL" />
-      </geometry>
-      <material name="carrier_black" />
-    </visual>
-    <collision>
-      <origin xyz="-0.39 0 0" rpy="0 1.5707963267949 0" />
-      <geometry>
-        <cylinder radius="${dock_arm_collision_radius}" length="${dock_arm_collision_length}" />
-      </geometry>
-    </collision>
-  </link>
-  <joint name="arm_joint_3" type="revolute">
-    <origin xyz="2.58061469903853 0.821037736652904 -0.0923428786138167" rpy="0 0 -3.14158674425948" />
-    <parent link="docking_3" />
-    <child link="dock_arm_3" />
-    <axis xyz="-0.99999999998254 0 0" />
-    <limit lower="-0.78539816339" upper="0.78539816339" effort="200.0" velocity="1.0" />
-    <dynamics damping="50.0" friction="20.0" />
-  </joint>
-  <link name="docking_4">
-    <inertial>
-      <origin xyz="1.57325903320313 0.822636592430764 -0.0944039787894342" rpy="0 0 0" />
-      <mass value="0.0202336294869927" />
-      <inertia ixx="9.72507400857707E-07" ixy="-2.37554290260085E-20" ixz="1.13271025171526E-20" iyy="8.0553172643547E-06" iyz="3.78249840438577E-35" izz="8.0553172643547E-06" />
-    </inertial>
-    <visual>
-      <origin xyz="0 0 0" rpy="0 0 0" />
-      <geometry>
-        <mesh filename="file:///home/bargavan/cyclus/src/carrier_emrac/meshes/visual/docking_4.STL" />
-      </geometry>
-      <material name="carrier_black" />
-    </visual>
-    <collision>
-      <origin xyz="${docking_collision_origin_2}" rpy="0 0 0" />
-      <geometry>
-        <box size="${docking_collision_size}" />
-      </geometry>
-    </collision>
-  </link>
-  <joint name="docking_arm_4" type="fixed">
-    <origin xyz="-0.857617979778071 -0.686214402146105 -1.15890213114568" rpy="1.5707963267949 0 0" />
-    <parent link="base_link" />
-    <child link="docking_4" />
-    <axis xyz="0 0 0" />
-  </joint>
-  <link name="dock_arm_4">
-    <inertial>
-      <origin xyz="-1.13743235222051 0.000575836874332936 0.000407762481724361" rpy="0 0 0" />
-      <mass value="0.00150072453201743" />
-      <inertia ixx="5.71130983246695E-07" ixy="-2.220630166025E-12" ixz="3.73861273025674E-16" iyy="1.95347256031264E-07" iyz="6.32661442998097E-11" izz="3.76033847997012E-07" />
-    </inertial>
-    <visual>
-      <origin xyz="0 0 0" rpy="0 0 0" />
-      <geometry>
-        <mesh filename="file:///home/bargavan/cyclus/src/carrier_emrac/meshes/visual/dock_arm_4.STL" />
-      </geometry>
-      <material name="carrier_black" />
-    </visual>
-    <collision>
-      <origin xyz="-0.39 0 0" rpy="0 1.5707963267949 0" />
-      <geometry>
-        <cylinder radius="${dock_arm_collision_radius}" length="${dock_arm_collision_length}" />
-      </geometry>
-    </collision>
-  </link>
-  <joint name="arm_joint_4" type="revolute">
-    <origin xyz="0.468826677599663 0.82263659243076 -0.0944039787894324" rpy="0 0 -3.14158674425949" />
-    <parent link="docking_4" />
-    <child link="dock_arm_4" />
-    <axis xyz="0.99999999998254 0 0" />
-    <limit lower="-0.78539816339" upper="0.78539816339" effort="200.0" velocity="1.0" />
-    <dynamics damping="50.0" friction="20.0" />
-  </joint>
-  <link name="lift_plate_carrier">
-    <inertial>
-      <origin xyz="0 0 0" rpy="0 0 0" />
-      <mass value="0.1" />
-      <inertia ixx="0.001" ixy="0.0" ixz="0.0" iyy="0.001" iyz="0.0" izz="0.001" />
-    </inertial>
-  </link>
-  <link name="lift_plate">
-    <inertial>
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