Commit message: Colouring_update&Vehicle_addup

File: urdf/cyclus_integrated_system.urdf.xacro (robot description, xacro)
@@ -16,4 +16,10 @@
   <xacro:arg name="ground_rails_mount_y" default="-0.02" />
   <xacro:arg name="ground_rails_mount_z" default="0.5" />
+  <xacro:arg name="tesla_mount_x" default="1.6" />
+  <xacro:arg name="tesla_mount_y" default="2.2" />
+  <xacro:arg name="tesla_mount_z" default="0.6" />
+  <xacro:arg name="tesla_mount_roll" default="1.570796" />
+  <xacro:arg name="tesla_mount_pitch" default="0.0" />
+  <xacro:arg name="tesla_mount_yaw" default="0.0" />
   <xacro:arg name="emrac_axis_1_xyz" default="1,0,0" />
   <xacro:arg name="emrac_axis_2_xyz" default="0,0,-1" />
@@ -37,4 +43,8 @@
   <xacro:property name="ground_rails_collision_size" value="3.3853313599 2.1556440430 0.0588344116" />
   <xacro:property name="ground_rails_collision_z" value="0.0294172058" />
+  <xacro:property name="tesla_mesh_scale" value="0.001 0.001 0.001" />
+  <xacro:property name="tesla_mesh_origin_x" value="0.0" />
+  <xacro:property name="tesla_mesh_origin_y" value="0.0" />
+  <xacro:property name="tesla_mesh_origin_z" value="0.0" />
   <xacro:property name="structure_gap_mm_value" value="$(arg structure_gap_mm)" />
   <xacro:property name="stationary_z_offset_value" value="$(arg stationary_z_offset)" />
@@ -67,4 +77,5 @@
     link_name="stationary_structure_right"
     mesh_name="stationary_structure_right.STL"
+    material_name="rail_bronze"
     pose_y="${right_pose_y}"
     pose_z="${stationary_z_offset_value}"
@@ -81,4 +92,5 @@
     link_name="stationary_structure_left"
     mesh_name="stationary_structure_left.STL"
+    material_name="rail_bronze"
     pose_y="${left_pose_y}"
     pose_z="${stationary_z_offset_value}"
@@ -93,7 +105,13 @@
   <xacro:cyclus_ground_rails
     root_link="integrated_root"
+    link_name="ground_rails"
+    mesh_name="ground_rails.STL"
+    material_name="rail_bronze"
     mount_x="$(arg ground_rails_mount_x)"
     mount_y="$(arg ground_rails_mount_y)"
     mount_z="$(arg ground_rails_mount_z)"
+    mount_roll="0"
+    mount_pitch="0"
+    mount_yaw="0"
     ground_rails_origin_x="${ground_rails_origin_x}"
     ground_rails_origin_y="${ground_rails_origin_y}"
@@ -102,4 +120,22 @@
     ground_rails_collision_size="${ground_rails_collision_size}"
     ground_rails_collision_z="${ground_rails_collision_z}" />
+  <xacro:cyclus_visual_mesh
+    root_link="integrated_root"
+    link_name="tesla_electric_vehicle"
+    mesh_name="tesla_electric_vehicle.STL"
+    material_name="cybertruck_steel"
+    mount_x="$(arg tesla_mount_x)"
+    mount_y="$(arg tesla_mount_y)"
+    mount_z="$(arg tesla_mount_z)"
+    mount_roll="$(arg tesla_mount_roll)"
+    mount_pitch="$(arg tesla_mount_pitch)"
+    mount_yaw="$(arg tesla_mount_yaw)"
+    mesh_origin_x="${tesla_mesh_origin_x}"
+    mesh_origin_y="${tesla_mesh_origin_y}"
+    mesh_origin_z="${tesla_mesh_origin_z}"
+    mesh_roll="0"
+    mesh_pitch="0"
+    mesh_yaw="0"
+    mesh_scale="${tesla_mesh_scale}" />
   <xacro:emrac_planar_mount prefix="emrac_1_" mount_x="${emrac_mount_x_value}" mount_y="${emrac_mount_y_value}" mount_z="${float(emrac_mount_z_value) + 0.0}" axis_1_vector="${emrac_axis_1_vector}" axis_2_vector="${emrac_axis_2_vector}" axis_1_limit="${emrac_axis_1_limit}" axis_2_limit="${emrac_axis_2_limit}" />
   <xacro:emrac_planar_mount prefix="emrac_2_" mount_x="${emrac_mount_x_value}" mount_y="${emrac_mount_y_value}" mount_z="${float(emrac_mount_z_value) + float(emrac_stack_z_step_value)}" axis_1_vector="${emrac_axis_1_vector}" axis_2_vector="${emrac_axis_2_vector}" axis_1_limit="${emrac_axis_1_limit}" axis_2_limit="${emrac_axis_2_limit}" />

File: urdf/emrac_body_macro.xacro (robot description, xacro)
@@ -59,5 +59,5 @@
         <mesh filename="file://$(find cyclus_description)/meshes/carrier_emrac/visual/docking_1.STL" />
       </geometry>
-      <material name="carrier_black" />
+      <material name="carrier_blue" />
     </visual>
     <collision>
@@ -85,5 +85,5 @@
         <mesh filename="file://$(find cyclus_description)/meshes/carrier_emrac/visual/dock_arm_1.STL" />
       </geometry>
-      <material name="carrier_black" />
+      <material name="rail_bronze" />
     </visual>
     <collision>
@@ -113,5 +113,5 @@
         <mesh filename="file://$(find cyclus_description)/meshes/carrier_emrac/visual/docking_2.STL" />
       </geometry>
-      <material name="carrier_black" />
+      <material name="carrier_blue" />
     </visual>
     <collision>
@@ -139,5 +139,5 @@
         <mesh filename="file://$(find cyclus_description)/meshes/carrier_emrac/visual/dock_arm_2.STL" />
       </geometry>
-      <material name="carrier_black" />
+      <material name="rail_bronze" />
     </visual>
     <collision>
@@ -167,5 +167,5 @@
         <mesh filename="file://$(find cyclus_description)/meshes/carrier_emrac/visual/docking_3.STL" />
       </geometry>
-      <material name="carrier_black" />
+      <material name="carrier_blue" />
     </visual>
     <collision>
@@ -193,5 +193,5 @@
         <mesh filename="file://$(find cyclus_description)/meshes/carrier_emrac/visual/dock_arm_3.STL" />
       </geometry>
-      <material name="carrier_black" />
+      <material name="rail_bronze" />
     </visual>
     <collision>
@@ -221,5 +221,5 @@
         <mesh filename="file://$(find cyclus_description)/meshes/carrier_emrac/visual/docking_4.STL" />
       </geometry>
-      <material name="carrier_black" />
+      <material name="carrier_blue" />
     </visual>
     <collision>
@@ -247,5 +247,5 @@
         <mesh filename="file://$(find cyclus_description)/meshes/carrier_emrac/visual/dock_arm_4.STL" />
       </geometry>
-      <material name="carrier_black" />
+      <material name="rail_bronze" />
     </visual>
     <collision>
@@ -282,5 +282,5 @@
         <mesh filename="file://$(find cyclus_description)/meshes/emrac/EMRAC Lift Plate Dwn Pos 1.stl" scale="${lift_plate_scale}" />
       </geometry>
-      <material name="lift_plate_grey" />
+      <material name="rail_bronze" />
     </visual>
     <collision>
@@ -296,5 +296,5 @@
     <child link="${prefix}lift_plate_carrier"/>
     <axis xyz="0 -1 0" />
-    <limit lower="-${lift_plate_travel}" upper="${lift_plate_travel}" effort="1000.0" velocity="0.58" />
+    <limit lower="-${lift_plate_travel}" upper="${lift_plate_travel}" effort="1000.0" velocity="0.55" />
     <dynamics damping="1.0" friction="0.05" />
   </joint>
@@ -305,15 +305,12 @@
   </joint>
   <gazebo reference="${prefix}base_link">
-    <material>Gazebo/Grey</material>
     <gravity>false</gravity>
     <self_collide>false</self_collide>
   </gazebo>
   <gazebo reference="${prefix}docking_1">
-    <material>Gazebo/DarkGrey</material>
     <gravity>false</gravity>
     <self_collide>false</self_collide>
   </gazebo>
   <gazebo reference="${prefix}dock_arm_1">
-    <material>Gazebo/DarkGrey</material>
     <gravity>false</gravity>
     <self_collide>false</self_collide>
@@ -322,10 +319,8 @@
   </gazebo>
   <gazebo reference="${prefix}docking_2">
-    <material>Gazebo/DarkGrey</material>
     <gravity>false</gravity>
     <self_collide>false</self_collide>
   </gazebo>
   <gazebo reference="${prefix}dock_arm_2">
-    <material>Gazebo/DarkGrey</material>
     <gravity>false</gravity>
     <self_collide>false</self_collide>
@@ -334,10 +329,8 @@
   </gazebo>
   <gazebo reference="${prefix}docking_3">
-    <material>Gazebo/DarkGrey</material>
     <gravity>false</gravity>
     <self_collide>false</self_collide>
   </gazebo>
   <gazebo reference="${prefix}dock_arm_3">
-    <material>Gazebo/DarkGrey</material>
     <gravity>false</gravity>
     <self_collide>false</self_collide>
@@ -346,10 +339,8 @@
   </gazebo>
   <gazebo reference="${prefix}docking_4">
-    <material>Gazebo/DarkGrey</material>
     <gravity>false</gravity>
     <self_collide>false</self_collide>
   </gazebo>
   <gazebo reference="${prefix}dock_arm_4">
-    <material>Gazebo/DarkGrey</material>
     <gravity>false</gravity>
     <self_collide>false</self_collide>
@@ -362,5 +353,4 @@
   </gazebo>
   <gazebo reference="${prefix}lift_plate">
-    <material>Gazebo/LightGrey</material>
     <gravity>false</gravity>
     <self_collide>false</self_collide>

File: urdf/includes/common_materials.xacro (robot description, xacro)
@@ -8,14 +8,27 @@
   <xacro:macro name="cyclus_shared_materials">
     <material name="steel_frame">
-      <color rgba="0.25 0.25 0.25 1.0" />
+      <color rgba="0.28 0.31 0.34 1.0" />
+    </material>
+    <material name="rail_bronze">
+      <color rgba="0.38 0.23 0.12 1.0" />
     </material>
     <material name="carrier_charcoal">
-      <color rgba="0.36 0.38 0.40 1.0" />
+      <color rgba="0.10 0.45 0.90 1.0" />
+    </material>
+    <material name="carrier_blue">
+      <color rgba="0.16 0.31 0.70 1.0" />
     </material>
     <material name="carrier_black">
-      <color rgba="0.24 0.25 0.27 1.0" />
+      <color rgba="0.10 0.45 0.90 1.0" />
+    </material>
+    <material name="tesla_red">
+      <color rgba="0.72 0.08 0.11 1.0" />
     </material>
     <material name="lift_plate_grey">
-      <color rgba="0.78 0.78 0.76 1.0" />
+      <color rgba="0.84 0.85 0.83 1.0" />
+    </material>
+    <!-- Cybertruck Stainless Steel -->
+    <material name="cybertruck_steel">
+      <color rgba="0.28 0.29 0.31 1.0" />
     </material>
   </xacro:macro>

File: urdf/includes/stationary_components.xacro (robot description, xacro)
@@ -6,5 +6,5 @@
 -->
 <robot xmlns:xacro="http://www.ros.org/wiki/xacro">
-  <xacro:macro name="cyclus_stationary_structure" params="root_link link_name mesh_name pose_y pose_z pose_yaw mesh_origin_x mesh_origin_y mesh_origin_z mesh_scale stationary_mesh_roll stationary_collision_size stationary_collision_z">
+  <xacro:macro name="cyclus_stationary_structure" params="root_link link_name mesh_name material_name pose_y pose_z pose_yaw mesh_origin_x mesh_origin_y mesh_origin_z mesh_scale stationary_mesh_roll stationary_collision_size stationary_collision_z">
     <link name="${link_name}">
       <inertial>
@@ -18,5 +18,5 @@
           <mesh filename="file://$(find cyclus_description)/meshes/${mesh_name}" scale="${mesh_scale}" />
         </geometry>
-        <material name="steel_frame" />
+        <material name="${material_name}" />
       </visual>
       <collision>
@@ -33,6 +33,6 @@
     </joint>
   </xacro:macro>
-  <xacro:macro name="cyclus_ground_rails" params="root_link mount_x mount_y mount_z ground_rails_origin_x ground_rails_origin_y ground_rails_origin_z mesh_scale ground_rails_collision_size ground_rails_collision_z">
-    <link name="ground_rails">
+  <xacro:macro name="cyclus_ground_rails" params="root_link link_name mesh_name material_name mount_x mount_y mount_z mount_roll mount_pitch mount_yaw ground_rails_origin_x ground_rails_origin_y ground_rails_origin_z mesh_scale ground_rails_collision_size ground_rails_collision_z">
+    <link name="${link_name}">
       <inertial>
         <origin xyz="0 0 0.03" rpy="0 0 0" />
@@ -43,7 +43,7 @@
         <origin xyz="${ground_rails_origin_x} ${ground_rails_origin_y} ${ground_rails_origin_z}" rpy="0 0 0" />
         <geometry>
-          <mesh filename="file://$(find cyclus_description)/meshes/ground_rails.STL" scale="${mesh_scale}" />
+          <mesh filename="file://$(find cyclus_description)/meshes/${mesh_name}" scale="${mesh_scale}" />
         </geometry>
-        <material name="steel_frame" />
+        <material name="${material_name}" />
       </visual>
       <collision>
@@ -54,8 +54,29 @@
       </collision>
     </link>
-    <joint name="${root_link}_to_ground_rails" type="fixed">
+    <joint name="${root_link}_to_${link_name}" type="fixed">
       <parent link="${root_link}" />
-      <child link="ground_rails" />
-      <origin xyz="${mount_x} ${mount_y} ${mount_z}" rpy="0 0 0" />
+      <child link="${link_name}" />
+      <origin xyz="${mount_x} ${mount_y} ${mount_z}" rpy="${mount_roll} ${mount_pitch} ${mount_yaw}" />
+    </joint>
+  </xacro:macro>
+  <xacro:macro name="cyclus_visual_mesh" params="root_link link_name mesh_name material_name mount_x mount_y mount_z mount_roll mount_pitch mount_yaw mesh_origin_x mesh_origin_y mesh_origin_z mesh_roll mesh_pitch mesh_yaw mesh_scale">
+    <link name="${link_name}">
+      <inertial>
+        <origin xyz="0 0 0" rpy="0 0 0" />
+        <mass value="10.0" />
+        <inertia ixx="1.0" ixy="0" ixz="0" iyy="1.0" iyz="0" izz="1.0" />
+      </inertial>
+      <visual>
+        <origin xyz="${mesh_origin_x} ${mesh_origin_y} ${mesh_origin_z}" rpy="${mesh_roll} ${mesh_pitch} ${mesh_yaw}" />
+        <geometry>
+          <mesh filename="file://$(find cyclus_description)/meshes/${mesh_name}" scale="${mesh_scale}" />
+        </geometry>
+        <material name="${material_name}" />
+      </visual>
+    </link>
+    <joint name="${root_link}_to_${link_name}" type="fixed">
+      <parent link="${root_link}" />
+      <child link="${link_name}" />
+      <origin xyz="${mount_x} ${mount_y} ${mount_z}" rpy="${mount_roll} ${mount_pitch} ${mount_yaw}" />
     </joint>
   </xacro:macro>
