Commit message: updated_colours_urdf

File: urdf/emrac_body_macro.xacro (robot description, xacro)
@@ -39,5 +39,5 @@
         <mesh filename="file://$(find cyclus_description)/meshes/carrier_emrac/visual/base_link.STL" />
       </geometry>
-      <material name="carrier_charcoal" />
+      <material name="emrac_body_grey" />
     </visual>
     <collision>
@@ -59,5 +59,5 @@
         <mesh filename="file://$(find cyclus_description)/meshes/carrier_emrac/visual/docking_1.STL" />
       </geometry>
-      <material name="carrier_blue" />
+      <material name="emrac_light_blue" />
     </visual>
     <collision>
@@ -85,5 +85,5 @@
         <mesh filename="file://$(find cyclus_description)/meshes/carrier_emrac/visual/dock_arm_1.STL" />
       </geometry>
-      <material name="rail_bronze" />
+      <material name="emrac_medium_grey" />
     </visual>
     <collision>
@@ -113,5 +113,5 @@
         <mesh filename="file://$(find cyclus_description)/meshes/carrier_emrac/visual/docking_2.STL" />
       </geometry>
-      <material name="carrier_blue" />
+      <material name="emrac_light_blue" />
     </visual>
     <collision>
@@ -139,5 +139,5 @@
         <mesh filename="file://$(find cyclus_description)/meshes/carrier_emrac/visual/dock_arm_2.STL" />
       </geometry>
-      <material name="rail_bronze" />
+      <material name="emrac_medium_grey" />
     </visual>
     <collision>
@@ -167,5 +167,5 @@
         <mesh filename="file://$(find cyclus_description)/meshes/carrier_emrac/visual/docking_3.STL" />
       </geometry>
-      <material name="carrier_blue" />
+      <material name="emrac_light_blue" />
     </visual>
     <collision>
@@ -193,5 +193,5 @@
         <mesh filename="file://$(find cyclus_description)/meshes/carrier_emrac/visual/dock_arm_3.STL" />
       </geometry>
-      <material name="rail_bronze" />
+      <material name="emrac_medium_grey" />
     </visual>
     <collision>
@@ -221,5 +221,5 @@
         <mesh filename="file://$(find cyclus_description)/meshes/carrier_emrac/visual/docking_4.STL" />
       </geometry>
-      <material name="carrier_blue" />
+      <material name="emrac_light_blue" />
     </visual>
     <collision>
@@ -247,5 +247,5 @@
         <mesh filename="file://$(find cyclus_description)/meshes/carrier_emrac/visual/dock_arm_4.STL" />
       </geometry>
-      <material name="rail_bronze" />
+      <material name="emrac_medium_grey" />
     </visual>
     <collision>
@@ -264,4 +264,137 @@
     <dynamics damping="50.0" friction="20.0" />
   </joint>
+  <link name="${prefix}wheels">
+    <inertial>
+      <origin xyz="0.4104 -0.83504 -0.26012" rpy="0 0 0" />
+      <mass value="66.927" />
+      <inertia ixx="0.31187" ixy="0.027609" ixz="0.0029563" iyy="11.966" iyz="0.0098157" izz="12.157" />
+    </inertial>
+    <visual>
+      <origin xyz="0 0 0" rpy="0 0 0" />
+      <geometry>
+        <mesh filename="file://$(find cyclus_description)/meshes/emrac_body_revised/visual/wheels.STL" />
+      </geometry>
+      <material name="professional_blue" />
+    </visual>
+    <collision>
+      <origin xyz="0 0 0" rpy="0 0 0" />
+      <geometry>
+        <mesh filename="file://$(find cyclus_description)/meshes/emrac_body_revised/collision/wheels.STL" />
+      </geometry>
+    </collision>
+  </link>
+  <joint name="${prefix}wheel_joint" type="fixed">
+    <origin xyz="-0.17912238382578 -0.989570036096044 0.451850726050984" rpy="1.5707963267949 0 0" />
+    <parent link="${prefix}base_link"/>
+    <child link="${prefix}wheels"/>
+  </joint>
+  <link name="${prefix}shaft_motors">
+    <inertial>
+      <origin xyz="2.1329 -0.83955 0.040521" rpy="0 0 0" />
+      <mass value="66.927" />
+      <inertia ixx="0.31187" ixy="0.027609" ixz="0.0029563" iyy="11.966" iyz="0.0098157" izz="12.157" />
+    </inertial>
+    <visual>
+      <origin xyz="0 0 0" rpy="0 0 0" />
+      <geometry>
+        <mesh filename="file://$(find cyclus_description)/meshes/emrac_body_revised/visual/shaft_motors.STL" />
+      </geometry>
+      <material name="deep_purple_semi">
+        <color rgba="0.30 0.12 0.45 0.8" />
+      </material>
+    </visual>
+    <collision>
+      <origin xyz="0 0 0" rpy="0 0 0" />
+      <geometry>
+        <mesh filename="file://$(find cyclus_description)/meshes/emrac_body_revised/collision/shaft_motors.STL" />
+      </geometry>
+    </collision>
+  </link>
+  <joint name="${prefix}shaft_motors_joint" type="fixed">
+    <origin xyz="-1.90167019372611 -0.688928868898414 0.456357618202888" rpy="1.5707963267949 0 0" />
+    <parent link="${prefix}base_link"/>
+    <child link="${prefix}shaft_motors"/>
+  </joint>
+  <link name="${prefix}shaft_pos">
+    <inertial>
+      <origin xyz="2.1329 -0.83955 0.040521" rpy="0 0 0" />
+      <mass value="66.927" />
+      <inertia ixx="0.31187" ixy="0.027609" ixz="0.0029563" iyy="11.966" iyz="0.0098157" izz="12.157" />
+    </inertial>
+    <visual>
+      <origin xyz="0 0 0" rpy="0 0 0" />
+      <geometry>
+        <mesh filename="file://$(find cyclus_description)/meshes/emrac_body_revised/visual/shaft_pos.STL" />
+      </geometry>
+      <material name="violet_semi">
+        <color rgba="0.58 0.40 0.74 0.7" />
+      </material>
+    </visual>
+    <collision>
+      <origin xyz="0 0 0" rpy="0 0 0" />
+      <geometry>
+        <mesh filename="file://$(find cyclus_description)/meshes/emrac_body_revised/collision/shaft_pos.STL" />
+      </geometry>
+    </collision>
+  </link>
+  <joint name="${prefix}shaft_pos_joint" type="fixed">
+    <origin xyz="-1.90167019372611 -0.688928868898414 0.456357618202888" rpy="1.5707963267949 0 0" />
+    <parent link="${prefix}base_link"/>
+    <child link="${prefix}shaft_pos"/>
+  </joint>
+  <link name="${prefix}support_block_pos">
+    <inertial>
+      <origin xyz="2.1329 -0.83955 0.040521" rpy="0 0 0" />
+      <mass value="66.927" />
+      <inertia ixx="0.31187" ixy="0.027609" ixz="0.0029563" iyy="11.966" iyz="0.0098157" izz="12.157" />
+    </inertial>
+    <visual>
+      <origin xyz="0 0 0" rpy="0 0 0" />
+      <geometry>
+        <mesh filename="file://$(find cyclus_description)/meshes/emrac_body_revised/visual/support_block_pos.STL" />
+      </geometry>
+      <material name="deep_red_semi">
+        <color rgba="0.55 0.08 0.08 0.6" />
+      </material>
+    </visual>
+    <collision>
+      <origin xyz="0 0 0" rpy="0 0 0" />
+      <geometry>
+        <mesh filename="file://$(find cyclus_description)/meshes/emrac_body_revised/collision/support_block_pos.STL" />
+      </geometry>
+    </collision>
+  </link>
+  <joint name="${prefix}suppott_block_joint" type="fixed">
+    <origin xyz="-1.90167019372611 -0.688928868898414 0.456357618202888" rpy="1.5707963267949 0 0" />
+    <parent link="${prefix}base_link"/>
+    <child link="${prefix}support_block_pos"/>
+  </joint>
+  <link name="${prefix}blots_pos">
+    <inertial>
+      <origin xyz="2.1329 -0.83955 0.040521" rpy="0 0 0" />
+      <mass value="66.927" />
+      <inertia ixx="0.31187" ixy="0.027609" ixz="0.0029563" iyy="11.966" iyz="0.0098157" izz="12.157" />
+    </inertial>
+    <visual>
+      <origin xyz="0 0 0" rpy="0 0 0" />
+      <geometry>
+        <mesh filename="file://$(find cyclus_description)/meshes/emrac_body_revised/visual/blots_pos.STL" />
+      </geometry>
+      <material name="bright_orange_semi">
+        <color rgba="0.90 0.45 0.10 0.5" />
+      </material>
+    </visual>
+    <collision>
+      <origin xyz="0 0 0" rpy="0 0 0" />
+      <geometry>
+        <mesh filename="file://$(find cyclus_description)/meshes/emrac_body_revised/collision/blots_pos.STL" />
+      </geometry>
+    </collision>
+  </link>
+  <joint name="${prefix}blots_pos_joint" type="fixed">
+    <origin xyz="-1.90167019372611 -0.688928868898414 0.456357618202888" rpy="1.5707963267949 0 0" />
+    <parent link="${prefix}base_link"/>
+    <child link="${prefix}blots_pos"/>
+  </joint>
   <link name="${prefix}lift_plate_carrier">
     <inertial>

File: urdf/includes/common_materials.xacro (robot description, xacro)
@@ -28,8 +28,79 @@
       <color rgba="0.82 0.84 0.86 1.0" />
     </material>
+    <material name="emrac_body_grey">
+      <color rgba="0.52941 0.54902 0.54902 1.0" />
+    </material>
+    <material name="emrac_light_blue">
+      <color rgba="0.79216 0.81961 0.93333 1.0" />
+    </material>
+    <material name="emrac_medium_grey">
+      <color rgba="0.49804 0.49804 0.49804 1.0" />
+    </material>
     <!-- Cybertruck Stainless Steel -->
     <material name="cybertruck_steel">
       <color rgba="0.62 0.64 0.66 1.0" />
     </material>
+    <!-- Professional Colors for New Components -->
+    <material name="industrial_dark_grey">
+      <color rgba="0.25 0.25 0.25 1.0" />
+    </material>
+    <material name="professional_blue">
+      <color rgba="0.16 0.39 0.68 1.0" />
+    </material>
+    <material name="carbon_grey">
+      <color rgba="0.35 0.35 0.37 1.0" />
+    </material>
+    <material name="slate_dark">
+      <color rgba="0.28 0.32 0.36 1.0" />
+    </material>
+    <material name="metallic_charcoal">
+      <color rgba="0.31 0.32 0.33 1.0" />
+    </material>
+        <!-- Additional Standard Colors -->
+    <material name="industrial_red">
+      <color rgba="0.78 0.18 0.18 1.0" />
+    </material>
+    <material name="deep_red">
+      <color rgba="0.55 0.08 0.08 1.0" />
+    </material>
+    <material name="signal_green">
+      <color rgba="0.18 0.62 0.24 1.0" />
+    </material>
+    <material name="forest_green">
+      <color rgba="0.13 0.39 0.16 1.0" />
+    </material>
+    <material name="lime_green">
+      <color rgba="0.56 0.80 0.22 1.0" />
+    </material>
+    <material name="royal_purple">
+      <color rgba="0.42 0.24 0.60 1.0" />
+    </material>
+    <material name="deep_purple">
+      <color rgba="0.30 0.12 0.45 1.0" />
+    </material>
+    <material name="violet">
+      <color rgba="0.58 0.40 0.74 1.0" />
+    </material>
+    <material name="bright_orange">
+      <color rgba="0.90 0.45 0.10 1.0" />
+    </material>
+    <material name="warning_yellow">
+      <color rgba="0.95 0.82 0.18 1.0" />
+    </material>
+    <material name="sky_blue">
+      <color rgba="0.35 0.67 0.93 1.0" />
+    </material>
+    <material name="cyan_blue">
+      <color rgba="0.12 0.72 0.78 1.0" />
+    </material>
+    <material name="matte_black">
+      <color rgba="0.08 0.08 0.08 1.0" />
+    </material>
+    <material name="pure_white">
+      <color rgba="0.96 0.96 0.96 1.0" />
+    </material>
+    <material name="silver_metallic">
+      <color rgba="0.75 0.76 0.78 1.0" />
+    </material>
   </xacro:macro>
 </robot>
